File: lm386_one_sp_amp.kicad_pcb (KiCad board)
At the start: 2 copper layers, 17 parts, among them U1 LM386

Commit message: 配置を進める
Parts:
- moved R7 40.9 mm to (205.1, 87.0), turned to -90 degrees
- moved C7 34.1 mm to (196.2, 93.3), turned to -90 degrees
- moved C3 32.3 mm to (197.6, 70.5), turned to 0 degrees
- moved C4 24.2 mm to (186.7, 94.6)
- moved C6 22.3 mm to (194.4, 86.4), turned to 0 degrees
- moved R6 21.9 mm to (201.9, 82.5), turned to 180 degrees
- moved BT1 20.7 mm to (207.7, 81.3), turned to 0 degrees
- moved R1 19.5 mm to (172.7, 69.8)
- moved R2 19.5 mm to (172.7, 72.4)
- moved LS1 19.4 mm to (177.2, 97.8)
- moved R4 18.4 mm to (172.7, 83.8)
- moved R5 18.4 mm to (172.7, 86.4)
- moved U1 16.1 mm to (183.5, 78.7)
- moved C2 14.4 mm to (176.5, 64.8), turned to 180 degrees
- moved C1 13.3 mm to (172.2, 76.8)
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
Commit message: 配置を修正
Parts:
- added H1: MountingHole, MyLibrary:MountingHole_3.2mm_M3, F.Cu at (123.2, 80.8)
- added H2: MountingHole, MyLibrary:MountingHole_3.2mm_M3, F.Cu at (163.8, 80.9)
- added H3: MountingHole, MyLibrary:MountingHole_3.2mm_M3, F.Cu at (123.2, 118.1)
- added H4: MountingHole, MyLibrary:MountingHole_3.2mm_M3, F.Cu at (163.8, 118.1)
- added J10: ToLED, MyLibrary:PinHeader_1x01_P2.54mm_Vertical, F.Cu at (152.3, 98.6)
- added J11: VR1_2, MyLibrary:PinHeader_1x01_P2.54mm_Vertical, F.Cu at (123.3, 106.1)
- added J12: VR2_2, MyLibrary:PinHeader_1x01_P2.54mm_Vertical, F.Cu at (123.3, 110.2)
- added J13: VR3_1, MyLibrary:PinHeader_1x01_P2.54mm_Vertical, F.Cu at (137.0, 90.3)
- added J14: VR3_3, MyLibrary:PinHeader_1x01_P2.54mm_Vertical, F.Cu at (137.0, 94.1)
- added J2: IN1, MyLibrary:PinHeader_1x01_P2.54mm_Vertical, F.Cu at (122.5, 90.9)
- added J3: IN2, MyLibrary:PinHeader_1x01_P2.54mm_Vertical, F.Cu at (121.2, 94.7)
- added J4: ToSW, MyLibrary:PinHeader_1x01_P2.54mm_Vertical, F.Cu at (156.1, 98.6)
- added J6: IN3, MyLibrary:PinHeader_1x01_P2.54mm_Vertical, F.Cu at (121.2, 98.5)
- added J7: VR2_1, MyLibrary:PinHeader_1x01_P2.54mm_Vertical, F.Cu at (123.3, 102.3)
- added J8: VR1_1, MyLibrary:PinHeader_1x01_P2.54mm_Vertical, F.Cu at (122.4, 86.7)
- added J9: FromSW, MyLibrary:PinHeader_1x01_P2.54mm_Vertical, F.Cu at (148.5, 98.6)
- C1: footprint Capacitor_THT:C_Rect_L10.3mm_W5.0mm_P7.50mm_MKS4 -> MyLibrary:11.6_7.0_p7.5
- C6: footprint Capacitor_THT:C_Rect_L9.0mm_W4.0mm_P7.50mm_MKT -> MyLibrary:9.3_4.3_p7.5
- moved R3 50.7 mm to (133.9, 101.5)
- moved C5 50.4 mm to (141.5, 89.0)
- moved C3 50.4 mm to (151.0, 89.7)
- moved C4 50.3 mm to (140.2, 113.8)
- moved C7 50.3 mm to (149.7, 112.5)
- moved R1 50.3 mm to (126.2, 89.0)
- moved R6 50.3 mm to (155.4, 101.7)
- moved U1 50.3 mm to (137.0, 97.9)
- moved BT1 50.3 mm to (161.2, 100.5)
- moved R2 50.3 mm to (126.2, 91.6)
- moved R7 50.3 mm to (158.6, 106.2)
- moved LS1 50.0 mm to (130.7, 116.3)
- moved C1 47.2 mm to (129.3, 96.5)
- moved C2 47.0 mm to (133.9, 84.6)
- moved C6 46.8 mm to (151.6, 105.5)
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Routing:
- net GND: track 0.00 -> 86.2 mm
- net Net-(C7-Pad2): track 0.00 -> 20.5 mm
- net Net-(J9-Pin_1): track 0.00 -> 17.1 mm
- net Net-(U1-BYPASS): track 0.00 -> 16.0 mm
- net Net-(J7-Pin_1): track 0.00 -> 12.2 mm
- net Net-(C6-Pad1): track 0.00 -> 11.0 mm
- net Net-(J8-Pin_1): track 0.00 -> 9.85 mm
- net Net-(C5-Pad2): track 0.00 -> 9.17 mm
- net Net-(U1-+): track 0.00 -> 7.06 mm
- net Net-(C2-Pad1): track 0.00 -> 6.98 mm
- net Net-(J3-Pin_1): track 0.00 -> 6.29 mm
- net Net-(BT1-+): track 0.00 -> 5.89 mm
- net Net-(D1-A): track 0.00 -> 5.61 mm
- net Net-(J13-Pin_1): track 0.00 -> 4.97 mm
- net Net-(J6-Pin_1): track 0.00 -> 4.54 mm
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- added copper zone on B.Cu, net GND
Other:
- board outline added: 50.3 x 47 mm
